Commit message: a1

File: urdf/autonet_v1.xacro (robot description, xacro)
@@ -6,9 +6,9 @@
   <link name="base_link">
     <!-- pose and inertial -->
-    <pose>0 0 0.05 0 0 0</pose>
+    <pose>-0.1 0 0.05 0 0 0</pose>
     <inertial>
       <mass value="5"/>
-      <origin rpy="0 0 0" xyz="0 0 0.05"/>
-      <inertia ixx="0.0395416666667" ixy="0" ixz="0" iyy="0.106208333333" iyz="0" izz="0.106208333333"/>
+      <origin rpy="0 0 0" xyz="-0.1 0 0.05"/>
+      <inertia ixx="0.106208333333" ixy="0" ixz="0" iyy="0.106208333333" iyz="0" izz="0.106208333333"/>
     </inertial>
     <!-- body -->
@@ -19,5 +19,5 @@
     </collision>
     <visual>
-      <origin rpy="0 0 0" xyz="0 0 0"/>
+      <origin rpy="0 0 0" xyz="-0.1 0 0"/>
       <geometry>
         <box size="0.295 0.295 0.05"/>
@@ -27,5 +27,5 @@
     <!-- caster front -->
     <collision name="caster_front_collision">]
-      <origin rpy="0 1.5707 0" xyz="-0.15 0 -0.012"/>
+      <origin rpy="0 1.5707 0" xyz="-0.25 0 -0.012"/>
       <geometry>
         <cylinder length="0.025" radius="0.038"/>
@@ -43,5 +43,5 @@
     </collision>
     <visual name="caster_front_visual">
-      <origin rpy="0 1.5707 0" xyz="0.15 0 -0.012"/>
+      <origin rpy="0 1.5707 0" xyz="-0.25 0 -0.012"/>
       <geometry>
         <cylinder length="0.025" radius="0.038"/>
@@ -76,6 +76,6 @@
    -->
   <xacro:link_wheel name="link_right_wheel" />
-  <xacro:joint_wheel name="joint_right_wheel" child="link_right_wheel" origin_xyz="-0.1 0.16 -0.012" />
+  <xacro:joint_wheel name="joint_right_wheel" child="link_right_wheel" origin_xyz="0 0.16 -0.012" />
   <xacro:link_wheel name="link_left_wheel" />
-  <xacro:joint_wheel name="joint_left_wheel" child="link_left_wheel" origin_xyz="-0.1 -0.16 -0.012" />
+  <xacro:joint_wheel name="joint_left_wheel" child="link_left_wheel" origin_xyz="0 -0.16 -0.012" />
 </robot>

File: urdf/macros.xacro (robot description, xacro)
@@ -29,5 +29,5 @@
         <axis rpy="0 0 0" xyz="0 1 0"/>
         <limit effort="10000" velocity="1000"/>
-        <joint_properties damping="1.0" friction="0.2"/>
+        <joint_properties damping="0" friction="0"/>
       </joint>
     </xacro:macro>

Commit message: SIMOK

File: urdf/autonet_v1.xacro (robot description, xacro)
@@ -8,7 +8,7 @@
     <pose>-0.1 0 0.05 0 0 0</pose>
     <inertial>
-      <mass value="5"/>
+      <mass value="0.5"/>
       <origin rpy="0 0 0" xyz="-0.1 0 0.05"/>
-      <inertia ixx="0.106208333333" ixy="0" ixz="0" iyy="0.106208333333" iyz="0" izz="0.106208333333"/>
+      <inertia ixx="0.206208333333" ixy="0" ixz="0" iyy="0.206208333333" iyz="0" izz="0.206208333333"/>
     </inertial>
     <!-- body -->

File: urdf/macros.xacro (robot description, xacro)
@@ -4,5 +4,5 @@
         <link name="${name}">
             <inertial>
-              <mass value="0.2"/>
+              <mass value="50"/>
               <origin rpy="0 1.5707 1.5707" xyz="0 0 0"/>
               <inertia ixx="0.000526666666667" ixy="0" ixz="0" iyy="0.000526666666667" iyz="0" izz="0.001"/>

Commit message: cam

File: urdf/autonet_v1.xacro (robot description, xacro)
@@ -1,4 +1,5 @@
 <?xml version="1.0" ?>
-<robot name="autonet_v1" xmlns:xacro="http://www.ros.org/wiki/xacro">
+<robot name="autonet_v1"
+  xmlns:xacro="http://www.ros.org/wiki/xacro">
   <xacro:include filename="$(find autonet_sim)/urdf/materials.xacro" />
   <xacro:include filename="$(find autonet_sim)/urdf/autonet_v1.gazebo" />
@@ -79,3 +80,69 @@
   <xacro:link_wheel name="link_left_wheel" />
   <xacro:joint_wheel name="joint_left_wheel" child="link_left_wheel" origin_xyz="0 -0.16 -0.012" />
+  <joint name="camera_joint" type="fixed">
+    <axis xyz="0 1 0" />
+    <origin xyz="0 0 0.2" rpy="0 0.2 0"/>
+    <parent link="base_link"/>
+    <child link="camera_link"/>
+  </joint>
+  <!-- Camera -->
+  <link name="camera_link">
+    <collision>
+      <origin xyz="0 0 0" rpy="0 0 0"/>
+      <geometry>
+        <box size="0.04 0.04 0.04"/>
+      </geometry>
+    </collision>
+    <visual>
+      <origin xyz="0 0 0" rpy="0 0 0"/>
+      <geometry>
+        <box size="0.04 0.04 0.04"/>
+      </geometry>
+      <material name="red"/>
+    </visual>
+    <inertial>
+      <mass value="1e-5" />
+      <origin xyz="0 0 0" rpy="0 0 0"/>
+      <inertia ixx="1e-6" ixy="0" ixz="0" iyy="1e-6" iyz="0" izz="1e-6" />
+    </inertial>
+  </link>
+  <gazebo reference="camera_link">
+    <sensor type="camera" name="camera1">
+      <update_rate>30.0</update_rate>
+      <camera name="head">
+        <horizontal_fov>1.3962634</horizontal_fov>
+        <image>
+          <width>640</width>
+          <height>480</height>
+          <format>R8G8B8</format>
+        </image>
+        <clip>
+          <near>0.02</near>
+          <far>300</far>
+        </clip>
+        <noise>
+          <type>gaussian</type>
+          <!-- Noise is sampled independently per pixel on each frame.
+               That pixel's noise value is added to each of its color
+               channels, which at that point lie in the range [0,1]. -->
+          <mean>0.0</mean>
+          <stddev>0.007</stddev>
+        </noise>
+      </camera>
+      <plugin name="camera_controller" filename="libgazebo_ros_camera.so">
+        <alwaysOn>true</alwaysOn>
+        <updateRate>0.0</updateRate>
+        <cameraName>camera1</cameraName>
+        <imageTopicName>image_raw</imageTopicName>
+        <cameraInfoTopicName>camera_info</cameraInfoTopicName>
+        <frameName>camera_link</frameName>
+        <hackBaseline>0.07</hackBaseline>
+        <distortionK1>0.0</distortionK1>
+        <distortionK2>0.0</distortionK2>
+        <distortionK3>0.0</distortionK3>
+        <distortionT1>0.0</distortionT1>
+        <distortionT2>0.0</distortionT2>
+      </plugin>
+    </sensor>
+  </gazebo>
 </robot>

Commit message: Robot stop bug and launch file

File: urdf/autonet_v1.xacro (robot description, xacro)
@@ -28,4 +28,26 @@
     <!-- caster front -->
     <collision name="caster_front_collision">]
+      <origin rpy="0 1.5707 0" xyz="0.05 0 -0.012"/>
+      <geometry>
+        <cylinder length="0.025" radius="0.038"/>
+      </geometry>
+      <surface>
+        <friction>
+          <ode>
+            <mu>0</mu>
+            <mu2>0</mu2>
+            <slip1>1.0</slip1>
+            <slip2>1.0</slip2>
+          </ode>
+        </friction>
+      </surface>
+    </collision>
+    <visual name="caster_front_visual">
+      <origin rpy="0 1.5707 0" xyz="0.05 0 -0.012"/>
+      <geometry>
+        <cylinder length="0.025" radius="0.038"/>
+      </geometry>
+    </visual>
+    <collision name="caster_back_collision">]
       <origin rpy="0 1.5707 0" xyz="-0.25 0 -0.012"/>
       <geometry>
@@ -43,5 +65,5 @@
       </surface>
     </collision>
-    <visual name="caster_front_visual">
+    <visual name="caster_back_visual">
       <origin rpy="0 1.5707 0" xyz="-0.25 0 -0.012"/>
       <geometry>

Commit message: tests

File: urdf/autonet_v1.xacro (robot description, xacro)
@@ -43,10 +43,10 @@
       </surface>
     </collision>
-    <visual name="caster_front_visual">
+    <!-- <visual name="caster_front_visual">
       <origin rpy="0 1.5707 0" xyz="0.05 0 -0.012"/>
       <geometry>
         <cylinder length="0.025" radius="0.038"/>
       </geometry>
-    </visual>
+    </visual> -->
     <collision name="caster_back_collision">]
       <origin rpy="0 1.5707 0" xyz="-0.25 0 -0.012"/>

Commit message: world with out buildings

File: urdf/autonet_v1.xacro (robot description, xacro)
@@ -104,5 +104,5 @@
   <joint name="camera_joint" type="fixed">
     <axis xyz="0 1 0" />
-    <origin xyz="0 0 0.2" rpy="0 0.2 0"/>
+    <origin xyz="0 -0.1 0.2" rpy="0 0.5 0"/>
     <parent link="base_link"/>
     <child link="camera_link"/>
@@ -133,5 +133,5 @@
       <update_rate>30.0</update_rate>
       <camera name="head">
-        <horizontal_fov>1.3962634</horizontal_fov>
+        <horizontal_fov>1.2262634</horizontal_fov>
         <image>
           <width>640</width>

Commit message: rename links

File: urdf/autonet_v1.xacro (robot description, xacro)
@@ -106,8 +106,8 @@
     <origin xyz="0 -0.1 0.2" rpy="0 0.5 0"/>
     <parent link="base_link"/>
-    <child link="camera_link"/>
+    <child link="camera1_link"/>
   </joint>
   <!-- Camera -->
-  <link name="camera_link">
+  <link name="camera1_link">
     <collision>
       <origin xyz="0 0 0" rpy="0 0 0"/>
@@ -129,5 +129,5 @@
     </inertial>
   </link>
-  <gazebo reference="camera_link">
+  <gazebo reference="camera1_link">
     <sensor type="camera" name="camera1">
       <update_rate>30.0</update_rate>
@@ -158,5 +158,5 @@
         <imageTopicName>image_raw</imageTopicName>
         <cameraInfoTopicName>camera_info</cameraInfoTopicName>
-        <frameName>camera_link</frameName>
+        <frameName>/camera1_link</frameName>
         <hackBaseline>0.07</hackBaseline>
         <distortionK1>0.0</distortionK1>
